Commit message: updated files

File: src/myrobot_description/urdf/v5_URDF.urdf (robot description, URDF)
Before this commit: robot myrobot_description, 22 links, 21 joints
Joints:
- joint f18: limit lower=0 upper=0.024 effort=0 velocity=0 -> lower=0 upper=0.024 effort=5.0 velocity=1.5
- joint f19: limit lower=-0.024 upper=0 effort=0 velocity=0 -> lower=-0.024 upper=0 effort=5.0 velocity=1.5
- joint f28: limit lower=-0.024 upper=0 effort=0 velocity=0 -> lower=-0.024 upper=0 effort=5.0 velocity=1.5
- joint f29: limit lower=0 upper=0.024 effort=0 velocity=0 -> lower=0 upper=0.024 effort=5.0 velocity=1.5
- joint j11: limit lower=-1.571 upper=1.571 effort=0 velocity=0 -> lower=-1.571 upper=1.571 effort=5.0 velocity=1.5
- joint j12: limit lower=-1.22 upper=0.105 effort=0 velocity=0 -> lower=-1.22 upper=0.105 effort=5.0 velocity=1.5
- joint j13: limit lower=-1.571 upper=1.571 effort=0 velocity=0 -> lower=-1.571 upper=1.571 effort=5.0 velocity=1.5
- joint j14: limit lower=-1.0472 upper=1.309 effort=0 velocity=0 -> lower=-1.0472 upper=1.309 effort=5.0 velocity=1.5
- joint j15: limit lower=-1.57 upper=1.57 effort=0 velocity=0 -> lower=-1.57 upper=1.57 effort=5.0 velocity=1.5
- joint j16: limit lower=-0.52 upper=0.52 effort=0 velocity=0 -> lower=-0.52 upper=0.52 effort=5.0 velocity=1.5
- joint j17: limit lower=-1.571 upper=1.571 effort=0 velocity=0 -> lower=-1.571 upper=1.571 effort=5.0 velocity=1.5
- joint j21: limit lower=-1.571 upper=1.571 effort=0 velocity=0 -> lower=-1.571 upper=1.571 effort=5.0 velocity=1.5
- joint j22: limit lower=-0.105 upper=1.22 effort=0 velocity=0 -> lower=-0.105 upper=1.22 effort=5.0 velocity=1.5
- joint j23: limit lower=-1.571 upper=1.571 effort=0 velocity=0 -> lower=-1.571 upper=1.571 effort=5.0 velocity=1.5
- joint j24: limit lower=-1.0472 upper=1.309 effort=0 velocity=0 -> lower=-1.0472 upper=1.309 effort=5.0 velocity=1.5
- joint j25: limit lower=-1.57 upper=1.57 effort=0 velocity=0 -> lower=-1.57 upper=1.57 effort=5.0 velocity=1.5
- joint j26: limit lower=-0.52 upper=0.52 effort=0 velocity=0 -> lower=-0.52 upper=0.52 effort=5.0 velocity=1.5
- joint j27: limit lower=-1.571 upper=1.571 effort=0 velocity=0 -> lower=-1.571 upper=1.571 effort=5.0 velocity=1.5
- joint j31: limit lower=-1.57 upper=1.57 effort=0 velocity=0 -> lower=-1.57 upper=1.57 effort=5.0 velocity=1.5
- joint j_32: limit lower=-0.52 upper=0.52 effort=0 velocity=0 -> lower=-0.52 upper=0.52 effort=5.0 velocity=1.5

Commit message: individual arm plan

File: src/myrobot_description/urdf/v5_URDF.urdf (robot description, URDF)
Before this commit: robot myrobot_description, 22 links, 21 joints
Joints:
- joint f18: limit lower=0 upper=0.024 effort=5.0 velocity=1.5 -> lower=0 upper=0.024 effort=0 velocity=0
- joint f19: limit lower=-0.024 upper=0 effort=5.0 velocity=1.5 -> lower=-0.024 upper=0 effort=0 velocity=0
- joint f28: limit lower=-0.024 upper=0 effort=5.0 velocity=1.5 -> lower=-0.024 upper=0 effort=0 velocity=0
- joint f29: limit lower=0 upper=0.024 effort=5.0 velocity=1.5 -> lower=0 upper=0.024 effort=0 velocity=0
- joint j11: limit lower=-1.571 upper=1.571 effort=5.0 velocity=1.5 -> lower=-1.571 upper=1.571 effort=0 velocity=0
- joint j12: limit lower=-1.22 upper=0.105 effort=5.0 velocity=1.5 -> lower=-1.22 upper=0.105 effort=0 velocity=0
- joint j13: limit lower=-1.571 upper=1.571 effort=5.0 velocity=1.5 -> lower=-1.571 upper=1.571 effort=0 velocity=0
- joint j14: limit lower=-1.0472 upper=1.309 effort=5.0 velocity=1.5 -> lower=-1.0472 upper=1.309 effort=0 velocity=0
- joint j15: limit lower=-1.57 upper=1.57 effort=5.0 velocity=1.5 -> lower=-1.57 upper=1.57 effort=0 velocity=0
- joint j16: limit lower=-0.52 upper=0.52 effort=5.0 velocity=1.5 -> lower=-0.52 upper=0.52 effort=0 velocity=0
- joint j17: limit lower=-1.571 upper=1.571 effort=5.0 velocity=1.5 -> lower=-1.571 upper=1.571 effort=0 velocity=0
- joint j21: limit lower=-1.571 upper=1.571 effort=5.0 velocity=1.5 -> lower=-1.571 upper=1.571 effort=0 velocity=0
- joint j22: limit lower=-0.105 upper=1.22 effort=5.0 velocity=1.5 -> lower=-0.105 upper=1.22 effort=0 velocity=0
- joint j23: limit lower=-1.571 upper=1.571 effort=5.0 velocity=1.5 -> lower=-1.571 upper=1.571 effort=0 velocity=0
- joint j24: limit lower=-1.0472 upper=1.309 effort=5.0 velocity=1.5 -> lower=-1.0472 upper=1.309 effort=0 velocity=0
- joint j25: limit lower=-1.57 upper=1.57 effort=5.0 velocity=1.5 -> lower=-1.57 upper=1.57 effort=0 velocity=0
- joint j26: limit lower=-0.52 upper=0.52 effort=5.0 velocity=1.5 -> lower=-0.52 upper=0.52 effort=0 velocity=0
- joint j27: limit lower=-1.571 upper=1.571 effort=5.0 velocity=1.5 -> lower=-1.571 upper=1.571 effort=0 velocity=0
- joint j31: limit lower=-1.57 upper=1.57 effort=5.0 velocity=1.5 -> lower=-1.57 upper=1.57 effort=0 velocity=0
- joint j_32: limit lower=-0.52 upper=0.52 effort=5.0 velocity=1.5 -> lower=-0.52 upper=0.52 effort=0 velocity=0
