Commit message: generate moveit config with newew urdf

File: src/myrobot_description/urdf/v2.urdf (robot description, URDF)
Before this commit: robot myrobot_description, 22 links, 21 joints
Links:
- added link TCP_Left, mass 0.044249; collision mesh filename=package://myrobot_description/meshes/TCP_Left.STL; visual mesh filename=package://myrobot_description/meshes/TCP_Left.STL
- added link TCP_right, mass 0.044249; collision mesh filename=package://myrobot_description/meshes/TCP_right.STL; visual mesh filename=package://myrobot_description/meshes/TCP_right.STL
- link base_link: mass 5.9028025886278 -> 5.9028
- link camera: mass 1.2669 -> 1.2668823887858
- link left_elbow_1: mass 0.164627752012669 -> 0.16463
- link left_elbow_2: mass 0.244439210733274 -> 0.24444
- link left_finger_1: mass 0.0609022601784627 -> 0.0609022601784625
- link left_finger_2: mass 0.0609022599124918 -> 0.060902
- link left_shoulder_1: mass 0.358791437962765 -> 0.358782813844843
- link left_shoulder_2: mass 0.0788967646315721 -> 0.0788967649028279
- link left_shoulder_3: mass 0.401297766857032 -> 0.401297704857678
- link left_wrist_1: mass 0.0180647810553896 -> 0.0180647810553899
- link left_wrist_2: mass 0.207514061526763 -> 0.207514061526779
- link neck_pitch: mass 0.78791 -> 0.787905683224849
- link neck_yaw: mass 0.02475 -> 5.9028
- link right_elbow_1: mass 0.164684756558366 -> 0.164684761985467
- link right_elbow_2: mass 0.237392378321504 -> 0.237392410184954
- link right_finger_1: mass 0.0609022599124917 -> 0.060902
- link right_finger_2: mass 0.0609022599124919 -> 0.060902
- link right_shoulder_1: mass 0.358747412616118 -> 0.35875
- link right_shoulder_2: mass 0.0788967649028125 -> 0.078897
- link right_shoulder_3: mass 0.401306132014166 -> 0.401304711733058
- link right_wrist_1: mass 0.0225938557953762 -> 0.022594
- link right_wrist_2: mass 0.20298498678678 -> 0.202984986786786
Joints:
- added joint f20: type fixed, parent right_wrist_2, child TCP_right, origin xyz=0.0011999 -0.15225 0.0001 rpy=0 0 0, axis 0 0 0
- added joint f30: type fixed, parent left_wrist_2, child TCP_Left, origin xyz=0.0015932 -0.14225 -2.7322E-05 rpy=0 0 0, axis 0 0 0
- joint f18: origin xyz=-0.0472293186770806 -0.0797999999999117 0.012800000000167 rpy=0 0 3.14159265358979 -> xyz=-0.047229 -0.0798 0.0128 rpy=0 0 3.1416
- joint f19: mimic (none) -> joint=f18 multiplier=-1 offset=0; origin xyz=0.0480618808715608 -0.0797999999999758 -0.0127999999994104 rpy=3.14159265358979 0 0 -> xyz=0.048062 -0.0798 -0.0128 rpy=3.1416 0 0
- joint f28: origin xyz=0.048429203299978 -0.0798000000000137 -0.012727322450562 rpy=-3.14159265358978 0 0 -> xyz=0.048429 -0.0798 -0.012727 rpy=-3.1416 0 0
- joint f29: limit lower=0 upper=0.024 effort=0 velocity=0 -> lower=-0.024 upper=0 effort=0 velocity=0; mimic (none) -> joint=f28 multiplier=-1 offset=0; origin xyz=-0.0468360049026447 -0.0798000000000124 0.0126726775494417 rpy=0 0 3.14159265358979 -> xyz=-0.046836 -0.0798 0.012673 rpy=0 0 3.1416
- joint j11: origin xyz=0 -0.206244975000007 -0.0122500000000135 rpy=1.5707963267949 0 3.14159265358979 -> xyz=0 -0.20624 -0.01225 rpy=1.5708 0 3.1416
- joint j12: limit lower=-1.22 upper=0.105 effort=0 velocity=0 -> lower=-2.269 upper=0.105 effort=0 velocity=0; origin xyz=0 0.000324623368866475 -0.0970303585666253 rpy=-1.5707963267949 -1.57015699455256 1.5707963267949 -> xyz=0 0.00032462 -0.09703 rpy=-1.5708 -1.5702 1.5708
- joint j13: axis 0 0.999999182508679 -0.00127866413627633 -> 0 1 -0.0012787; origin xyz=-0.000197322450632975 -0.0552057468871058 0.00797500000025222 rpy=0.00127866448471928 1.5707963267949 0 -> xyz=-0.00019732 -0.055206 0.007975 rpy=0.0012787 1.5708 0
- joint j15: origin xyz=-1.83717277871809E-05 0.101985602391172 0.00019732244229459 rpy=3.14159265358979 0 3.14159265358979 -> xyz=-1.8372E-05 0.10199 0.00019732 rpy=3.1416 0 3.1416
- joint j16: axis -0.999999795627149 -0.000639332198812096 0 -> -1 -0.00063933 0; limit lower=-0.52 upper=0.52 effort=0 velocity=0 -> lower=-0.95993 upper=1.5533 effort=0 velocity=0; origin xyz=0.000338552314752161 0.147652253083333 0.000497322442299319 rpy=0 0 3.14095332134742 -> xyz=0.00033855 0.14765 0.00049732 rpy=0 0 3.141
- joint j17: origin xyz=0.000494644890471518 -0.0450001174205644 -0.000127322447598478 rpy=0 0 0 -> xyz=0.00049464 -0.045 -0.00012732 rpy=0 0 0
- joint j21: origin xyz=0 0.206244974999998 -0.012250000000019 rpy=1.5707963267949 0 3.14159265358979 -> xyz=0 0.20624 -0.01225 rpy=1.5708 0 3.1416
- joint j22: limit lower=-0.105 upper=1.22 effort=0 velocity=0 -> lower=-0.105 upper=2.269 effort=0 velocity=0; origin xyz=0 0.000324623368871669 0.0970303585666364 rpy=0 -1.5707963267949 0 -> xyz=0 0.00032462 0.09703 rpy=0 -1.5708 0
- joint j23: origin xyz=0.000197322450478765 -0.0552026775494689 0.00797500000000062 rpy=1.57079632679491 0 3.14159265358979 -> xyz=0.00019732 -0.055203 0.007975 rpy=1.5708 0 3.1416
- joint j24: origin xyz=0 -0.000199999999985666 -0.224700000000006 rpy=1.5707963267949 1.5707963267949 0 -> xyz=0 -0.0002 -0.2247 rpy=1.5708 1.5708 0
- joint j25: origin xyz=0.0975853550987641 0.000297322450554638 0.000197322450540465 rpy=0 0 -1.5707963267949 -> xyz=0.097585 0.00029732 0.00019732 rpy=0 0 -1.5708
- joint j26: limit lower=-0.52 upper=0.52 effort=0 velocity=0 -> lower=-0.95993 upper=1.5533 effort=0 velocity=0; origin xyz=0 0.152052677549566 -0.000297322450548531 rpy=0 0 -3.14159265358979 -> xyz=0 0.15205 -0.00029732 rpy=0 0 -3.1416
- joint j27: origin xyz=0.000127322450572731 -0.0449999999999919 0 rpy=0 0 0 -> xyz=0.00012732 -0.045 0 rpy=0 0 0
- joint j31: limit lower=-1.57 upper=1.57 effort=0 velocity=0 -> (none); origin xyz=0.00875 0 0.1486 rpy=1.5708 0 1.5708 -> xyz=0.00874999999999426 0 0.148599999999878 rpy=1.5707963267949 0 1.5707963267949; type revolute -> continuous
- joint j_32: limit lower=-0.52 upper=0.52 effort=0 velocity=0 -> (none); type revolute -> continuous

Commit message: gripper joint limits fix

File: src/myrobot_description/urdf/v2.urdf (robot description, URDF)
Before this commit: robot v2, 24 links, 23 joints
Joints:
- joint f29: limit lower=-0.024 upper=0 effort=0 velocity=0 -> lower=0 upper=+0.024 effort=0 velocity=0

Commit message: urdf limit update

File: src/myrobot_description/urdf/v2.urdf (robot description, URDF)
Before this commit: robot v2, 24 links, 23 joints
Joints:
- joint f29: limit lower=0 upper=+0.024 effort=0 velocity=0 -> lower=0 upper=0.024 effort=0 velocity=0
- joint j12: limit lower=-2.269 upper=0.105 effort=0 velocity=0 -> lower=-1.22 upper=0.105 effort=0 velocity=0
- joint j16: limit lower=-0.95993 upper=1.5533 effort=0 velocity=0 -> lower=-0.52 upper=0.52 effort=0 velocity=0
- joint j22: limit lower=-0.105 upper=2.269 effort=0 velocity=0 -> lower=-0.105 upper=1.22 effort=0 velocity=0
- joint j26: limit lower=-0.95993 upper=1.5533 effort=0 velocity=0 -> lower=-0.52 upper=0.52 effort=0 velocity=0
- joint j31: limit (none) -> lower=-1.57 upper=1.57 effort=0 velocity=0
- joint j_32: limit (none) -> lower=-0.52 upper=0.52 effort=0 velocity=0

Commit message: plan and execute using individual joint degrees in rviz

File: src/myrobot_description/urdf/v2.urdf (robot description, URDF)
Before this commit: robot v2, 24 links, 23 joints
Links:
- link base_link: mass 5.9028 -> 5.9028025886278
- link camera: mass 1.2668823887858 -> 1.2669
- link left_elbow_1: mass 0.16463 -> 0.164627752012669
- link left_elbow_2: mass 0.24444 -> 0.244439210733274
- link left_finger_1: mass 0.0609022601784625 -> 0.0609022601784627
- link left_finger_2: mass 0.060902 -> 0.0609022599124918
- link left_shoulder_1: mass 0.358782813844843 -> 0.358791437962765
- link left_shoulder_2: mass 0.0788967649028279 -> 0.0788967646315721
- link left_shoulder_3: mass 0.401297704857678 -> 0.401297766857032
- link left_wrist_1: mass 0.0180647810553899 -> 0.0180647810553896
- link left_wrist_2: mass 0.207514061526779 -> 0.207514061526763
- link neck_pitch: mass 0.787905683224849 -> 0.78791
- link neck_yaw: mass 5.9028 -> 0.02475
- link right_elbow_1: mass 0.164684761985467 -> 0.164684756558366
- link right_elbow_2: mass 0.237392410184954 -> 0.237392378321504
- link right_finger_1: mass 0.060902 -> 0.0609022599124917
- link right_finger_2: mass 0.060902 -> 0.0609022599124919
- link right_shoulder_1: mass 0.35875 -> 0.358747412616118
- link right_shoulder_2: mass 0.078897 -> 0.0788967649028125
- link right_shoulder_3: mass 0.401304711733058 -> 0.401306132014166
- link right_wrist_1: mass 0.022594 -> 0.0225938557953762
- link right_wrist_2: mass 0.202984986786786 -> 0.20298498678678
Joints:
- joint f18: origin xyz=-0.047229 -0.0798 0.0128 rpy=0 0 3.1416 -> xyz=-0.0472293186770806 -0.0797999999999117 0.012800000000167 rpy=0 0 3.14159265358979
- joint f19: origin xyz=0.048062 -0.0798 -0.0128 rpy=3.1416 0 0 -> xyz=0.0480618808715608 -0.0797999999999758 -0.0127999999994104 rpy=3.14159265358979 0 0
- joint f28: origin xyz=0.048429 -0.0798 -0.012727 rpy=-3.1416 0 0 -> xyz=0.048429203299978 -0.0798000000000137 -0.012727322450562 rpy=-3.14159265358978 0 0
- joint f29: origin xyz=-0.046836 -0.0798 0.012673 rpy=0 0 3.1416 -> xyz=-0.0468360049026447 -0.0798000000000124 0.0126726775494417 rpy=0 0 3.14159265358979
- joint j11: origin xyz=0 -0.20624 -0.01225 rpy=1.5708 0 3.1416 -> xyz=0 -0.206244975000007 -0.0122500000000135 rpy=1.5707963267949 0 3.14159265358979
- joint j12: origin xyz=0 0.00032462 -0.09703 rpy=-1.5708 -1.5702 1.5708 -> xyz=0 0.000324623368866475 -0.0970303585666253 rpy=-1.5707963267949 -1.57015699455256 1.5707963267949
- joint j13: axis 0 1 -0.0012787 -> 0 0.999999182508679 -0.00127866413627633; origin xyz=-0.00019732 -0.055206 0.007975 rpy=0.0012787 1.5708 0 -> xyz=-0.000197322450632975 -0.0552057468871058 0.00797500000025222 rpy=0.00127866448471928 1.5707963267949 0
- joint j15: origin xyz=-1.8372E-05 0.10199 0.00019732 rpy=3.1416 0 3.1416 -> xyz=-1.83717277871809E-05 0.101985602391172 0.00019732244229459 rpy=3.14159265358979 0 3.14159265358979
- joint j16: axis -1 -0.00063933 0 -> -0.999999795627149 -0.000639332198812096 0; origin xyz=0.00033855 0.14765 0.00049732 rpy=0 0 3.141 -> xyz=0.000338552314752161 0.147652253083333 0.000497322442299319 rpy=0 0 3.14095332134742
- joint j17: origin xyz=0.00049464 -0.045 -0.00012732 rpy=0 0 0 -> xyz=0.000494644890471518 -0.0450001174205644 -0.000127322447598478 rpy=0 0 0
- joint j21: origin xyz=0 0.20624 -0.01225 rpy=1.5708 0 3.1416 -> xyz=0 0.206244974999998 -0.012250000000019 rpy=1.5707963267949 0 3.14159265358979
- joint j22: origin xyz=0 0.00032462 0.09703 rpy=0 -1.5708 0 -> xyz=0 0.000324623368871669 0.0970303585666364 rpy=0 -1.5707963267949 0
- joint j23: origin xyz=0.00019732 -0.055203 0.007975 rpy=1.5708 0 3.1416 -> xyz=0.000197322450478765 -0.0552026775494689 0.00797500000000062 rpy=1.57079632679491 0 3.14159265358979
- joint j24: origin xyz=0 -0.0002 -0.2247 rpy=1.5708 1.5708 0 -> xyz=0 -0.000199999999985666 -0.224700000000006 rpy=1.5707963267949 1.5707963267949 0
- joint j25: origin xyz=0.097585 0.00029732 0.00019732 rpy=0 0 -1.5708 -> xyz=0.0975853550987641 0.000297322450554638 0.000197322450540465 rpy=0 0 -1.5707963267949
- joint j26: origin xyz=0 0.15205 -0.00029732 rpy=0 0 -3.1416 -> xyz=0 0.152052677549566 -0.000297322450548531 rpy=0 0 -3.14159265358979
- joint j27: origin xyz=0.00012732 -0.045 0 rpy=0 0 0 -> xyz=0.000127322450572731 -0.0449999999999919 0 rpy=0 0 0
- joint j31: origin xyz=0.00874999999999426 0 0.148599999999878 rpy=1.5707963267949 0 1.5707963267949 -> xyz=0.00875 0 0.1486 rpy=1.5708 0 1.5708; type continuous -> revolute
- joint j_32: type continuous -> revolute
