Commit message: xl actuators going wooooooo

File: src/myrobot_moveit_config/config/myrobot_description.ros2_control.xacro (robot description, xacro)
@@ -27,42 +27,46 @@
         <param name="error_timeout_sec">0.2</param>
         <param name="dynamixel_model_folder">/param/dxl_model</param>
-          <!-- 14 joints with 14 transmissions (each transmission drives a single joint) -->
-          <param name="number_of_joints">14</param>
-          <param name="number_of_transmissions">14</param>
-          <!-- transmission_to_joint_matrix is a 14x14 identity matrix -->
+          <!-- 16 joints with 16 transmissions (each transmission drives a single joint) -->
+          <param name="number_of_joints">16</param>
+          <param name="number_of_transmissions">16</param>
+          <!-- transmission_to_joint_matrix is a 16x16 identity matrix -->
           <!-- Each row: transmission i drives joint i -->
           <param name="transmission_to_joint_matrix">
-          1, 0, 0, 0, 0, 0, 0, 0, 0, 0, 0, 0, 0, 0,
-          0, 1, 0, 0, 0, 0, 0, 0, 0, 0, 0, 0, 0, 0,
-          0, 0, 1, 0, 0, 0, 0, 0, 0, 0, 0, 0, 0, 0,
-          0, 0, 0, 1, 0, 0, 0, 0, 0, 0, 0, 0, 0, 0,
-          0, 0, 0, 0, 1, 0, 0, 0, 0, 0, 0, 0, 0, 0,
-          0, 0, 0, 0, 0, 1, 0, 0, 0, 0, 0, 0, 0, 0,
-          0, 0, 0, 0, 0, 0, 1, 0, 0, 0, 0, 0, 0, 0,
-          0, 0, 0, 0, 0, 0, 0, 1, 0, 0, 0, 0, 0, 0,
-          0, 0, 0, 0, 0, 0, 0, 0, 1, 0, 0, 0, 0, 0,
-          0, 0, 0, 0, 0, 0, 0, 0, 0, 1, 0, 0, 0, 0,
-          0, 0, 0, 0, 0, 0, 0, 0, 0, 0, 1, 0, 0, 0,
-          0, 0, 0, 0, 0, 0, 0, 0, 0, 0, 0, 1, 0, 0,
-          0, 0, 0, 0, 0, 0, 0, 0, 0, 0, 0, 0, 1, 0,
-          0, 0, 0, 0, 0, 0, 0, 0, 0, 0, 0, 0, 0, 1
+          1, 0, 0, 0, 0, 0, 0, 0, 0, 0, 0, 0, 0, 0, 0, 0,
+          0, 1, 0, 0, 0, 0, 0, 0, 0, 0, 0, 0, 0, 0, 0, 0,
+          0, 0, 1, 0, 0, 0, 0, 0, 0, 0, 0, 0, 0, 0, 0, 0,
+          0, 0, 0, 1, 0, 0, 0, 0, 0, 0, 0, 0, 0, 0, 0, 0,
+          0, 0, 0, 0, 1, 0, 0, 0, 0, 0, 0, 0, 0, 0, 0, 0,
+          0, 0, 0, 0, 0, 1, 0, 0, 0, 0, 0, 0, 0, 0, 0, 0,
+          0, 0, 0, 0, 0, 0, 1, 0, 0, 0, 0, 0, 0, 0, 0, 0,
+          0, 0, 0, 0, 0, 0, 0, 1, 0, 0, 0, 0, 0, 0, 0, 0,
+          0, 0, 0, 0, 0, 0, 0, 0, 1, 0, 0, 0, 0, 0, 0, 0,
+          0, 0, 0, 0, 0, 0, 0, 0, 0, 1, 0, 0, 0, 0, 0, 0,
+          0, 0, 0, 0, 0, 0, 0, 0, 0, 0, 1, 0, 0, 0, 0, 0,
+          0, 0, 0, 0, 0, 0, 0, 0, 0, 0, 0, 1, 0, 0, 0, 0,
+          0, 0, 0, 0, 0, 0, 0, 0, 0, 0, 0, 0, 1, 0, 0, 0,
+          0, 0, 0, 0, 0, 0, 0, 0, 0, 0, 0, 0, 0, 1, 0, 0,
+          0, 0, 0, 0, 0, 0, 0, 0, 0, 0, 0, 0, 0, 0, 1, 0,
+          0, 0, 0, 0, 0, 0, 0, 0, 0, 0, 0, 0, 0, 0, 0, 1
           </param>
           <!-- joint_to_transmission_matrix is a 14x14 identity matrix -->
           <!-- Each joint is fully driven by its corresponding transmission -->
           <param name="joint_to_transmission_matrix">
-          1, 0, 0, 0, 0, 0, 0, 0, 0, 0, 0, 0, 0, 0,
-          0, 1, 0, 0, 0, 0, 0, 0, 0, 0, 0, 0, 0, 0,
-          0, 0, 1, 0, 0, 0, 0, 0, 0, 0, 0, 0, 0, 0,
-          0, 0, 0, 1, 0, 0, 0, 0, 0, 0, 0, 0, 0, 0,
-          0, 0, 0, 0, 1, 0, 0, 0, 0, 0, 0, 0, 0, 0,
-          0, 0, 0, 0, 0, 1, 0, 0, 0, 0, 0, 0, 0, 0,
-          0, 0, 0, 0, 0, 0, 1, 0, 0, 0, 0, 0, 0, 0,
-          0, 0, 0, 0, 0, 0, 0, 1, 0, 0, 0, 0, 0, 0,
-          0, 0, 0, 0, 0, 0, 0, 0, 1, 0, 0, 0, 0, 0,
-          0, 0, 0, 0, 0, 0, 0, 0, 0, 1, 0, 0, 0, 0,
-          0, 0, 0, 0, 0, 0, 0, 0, 0, 0, 1, 0, 0, 0,
-          0, 0, 0, 0, 0, 0, 0, 0, 0, 0, 0, 1, 0, 0,
-          0, 0, 0, 0, 0, 0, 0, 0, 0, 0, 0, 0, 1, 0,
-          0, 0, 0, 0, 0, 0, 0, 0, 0, 0, 0, 0, 0, 1
+          1, 0, 0, 0, 0, 0, 0, 0, 0, 0, 0, 0, 0, 0, 0, 0,
+          0, 1, 0, 0, 0, 0, 0, 0, 0, 0, 0, 0, 0, 0, 0, 0,
+          0, 0, 1, 0, 0, 0, 0, 0, 0, 0, 0, 0, 0, 0, 0, 0,
+          0, 0, 0, 1, 0, 0, 0, 0, 0, 0, 0, 0, 0, 0, 0, 0,
+          0, 0, 0, 0, 1, 0, 0, 0, 0, 0, 0, 0, 0, 0, 0, 0,
+          0, 0, 0, 0, 0, 1, 0, 0, 0, 0, 0, 0, 0, 0, 0, 0,
+          0, 0, 0, 0, 0, 0, 1, 0, 0, 0, 0, 0, 0, 0, 0, 0,
+          0, 0, 0, 0, 0, 0, 0, 1, 0, 0, 0, 0, 0, 0, 0, 0,
+          0, 0, 0, 0, 0, 0, 0, 0, 1, 0, 0, 0, 0, 0, 0, 0,
+          0, 0, 0, 0, 0, 0, 0, 0, 0, 1, 0, 0, 0, 0, 0, 0,
+          0, 0, 0, 0, 0, 0, 0, 0, 0, 0, 1, 0, 0, 0, 0, 0,
+          0, 0, 0, 0, 0, 0, 0, 0, 0, 0, 0, 1, 0, 0, 0, 0,
+          0, 0, 0, 0, 0, 0, 0, 0, 0, 0, 0, 0, 1, 0, 0, 0,
+          0, 0, 0, 0, 0, 0, 0, 0, 0, 0, 0, 0, 0, 1, 0, 0,
+          0, 0, 0, 0, 0, 0, 0, 0, 0, 0, 0, 0, 0, 0, 1, 0,
+          0, 0, 0, 0, 0, 0, 0, 0, 0, 0, 0, 0, 0, 0, 0, 1
           </param>
         <param name="ros_update_freq">200</param>
@@ -180,5 +184,5 @@
       </joint>
       <!-- Head Joints -->
-      <!-- <joint name="j31">
+      <joint name="j31">
         <command_interface name="position"/>
         <state_interface name="position">
@@ -193,5 +197,5 @@
         </state_interface>
         <state_interface name="velocity"/>
-      </joint> -->
+      </joint>
       <!-- GPIO Blocks for each dynamixel (IDs 0 to 15 for 16 joints) -->
       <gpio name="dxl1">
@@ -201,5 +205,5 @@
         <state_interface name="Present Position"/>
         <state_interface name="Present Velocity"/>
-        <state_interface name="Present Current"/>
+        <!-- <state_interface name="Present Current"/> -->
         <state_interface name="Torque Enable"/>
         <state_interface name="Present Input Voltage"/>
@@ -217,5 +221,5 @@
         <state_interface name="Present Position"/>
         <state_interface name="Present Velocity"/>
-        <state_interface name="Present Current"/>
+        <!-- <state_interface name="Present Current"/> -->
         <state_interface name="Torque Enable"/>
         <state_interface name="Present Input Voltage"/>
@@ -233,5 +237,5 @@
         <state_interface name="Present Position"/>
         <state_interface name="Present Velocity"/>
-        <state_interface name="Present Current"/>
+        <!-- <state_interface name="Present Current"/> -->
         <state_interface name="Torque Enable"/>
         <state_interface name="Present Input Voltage"/>
@@ -249,5 +253,5 @@
         <state_interface name="Present Position"/>
         <state_interface name="Present Velocity"/>
-        <state_interface name="Present Current"/>
+        <!-- <state_interface name="Present Current"/> -->
         <state_interface name="Torque Enable"/>
         <state_interface name="Present Input Voltage"/>
@@ -265,5 +269,5 @@
         <state_interface name="Present Position"/>
         <state_interface name="Present Velocity"/>
-        <state_interface name="Present Current"/>
+        <!-- <state_interface name="Present Current"/> -->
         <state_interface name="Torque Enable"/>
         <state_interface name="Present Input Voltage"/>
@@ -281,5 +285,5 @@
         <state_interface name="Present Position"/>
         <state_interface name="Present Velocity"/>
-        <state_interface name="Present Current"/>
+        <!-- <state_interface name="Present Current"/> -->
         <state_interface name="Torque Enable"/>
         <state_interface name="Present Input Voltage"/>
@@ -297,5 +301,5 @@
         <state_interface name="Present Position"/>
         <state_interface name="Present Velocity"/>
-        <state_interface name="Present Current"/>
+        <!-- <state_interface name="Present Current"/> -->
         <state_interface name="Torque Enable"/>
         <state_interface name="Present Input Voltage"/>
@@ -313,5 +317,5 @@
         <state_interface name="Present Position"/>
         <state_interface name="Present Velocity"/>
-        <state_interface name="Present Current"/>
+        <!-- <state_interface name="Present Current"/> -->
         <state_interface name="Torque Enable"/>
         <state_interface name="Present Input Voltage"/>
@@ -329,5 +333,5 @@
         <state_interface name="Present Position"/>
         <state_interface name="Present Velocity"/>
-        <state_interface name="Present Current"/>
+        <!-- <state_interface name="Present Current"/> -->
         <state_interface name="Torque Enable"/>
         <state_interface name="Present Input Voltage"/>
@@ -345,5 +349,5 @@
         <state_interface name="Present Position"/>
         <state_interface name="Present Velocity"/>
-        <state_interface name="Present Current"/>
+        <!-- <state_interface name="Present Current"/> -->
         <state_interface name="Torque Enable"/>
         <state_interface name="Present Input Voltage"/>
@@ -361,5 +365,5 @@
         <state_interface name="Present Position"/>
         <state_interface name="Present Velocity"/>
-        <state_interface name="Present Current"/>
+        <!-- <state_interface name="Present Current"/> -->
         <state_interface name="Torque Enable"/>
         <state_interface name="Present Input Voltage"/>
@@ -377,5 +381,5 @@
         <state_interface name="Present Position"/>
         <state_interface name="Present Velocity"/>
-        <state_interface name="Present Current"/>
+        <!-- <state_interface name="Present Current"/> -->
         <state_interface name="Torque Enable"/>
         <state_interface name="Present Input Voltage"/>
@@ -393,5 +397,5 @@
         <state_interface name="Present Position"/>
         <state_interface name="Present Velocity"/>
-        <state_interface name="Present Current"/>
+        <!-- <state_interface name="Present Current"/> -->
         <state_interface name="Torque Enable"/>
         <state_interface name="Present Input Voltage"/>
@@ -409,46 +413,46 @@
         <state_interface name="Present Position"/>
         <state_interface name="Present Velocity"/>
-        <state_interface name="Present Current"/>
-        <state_interface name="Torque Enable"/>
-        <state_interface name="Present Input Voltage"/>
-        <param name="Position P Gain">800</param>
-        <param name="Position I Gain">100</param>
-        <param name="Position D Gain">100</param>
-        <param name="Profile Velocity">200</param>
-        <param name="Profile Acceleration">50</param>
-        <param name="Drive Mode">0</param>
-      </gpio>
-      <!-- <gpio name="dxl15">
-        <param name="type">dxl</param>
-        <param name="ID">14</param>
-        <command_interface name="Goal Position"/>
-        <state_interface name="Present Position"/>
-        <state_interface name="Present Velocity"/>
-        <state_interface name="Present Current"/>
-        <state_interface name="Torque Enable"/>
-        <state_interface name="Present Input Voltage"/>
-        <param name="Position P Gain">800</param>
-        <param name="Position I Gain">100</param>
-        <param name="Position D Gain">100</param>
-        <param name="Profile Velocity">200</param>
-        <param name="Profile Acceleration">50</param>
-        <param name="Drive Mode">0</param>
+        <!-- <state_interface name="Present Current"/> -->
+        <state_interface name="Torque Enable"/>
+        <state_interface name="Present Input Voltage"/>
+        <param name="Position P Gain">800</param>
+        <param name="Position I Gain">100</param>
+        <param name="Position D Gain">100</param>
+        <param name="Profile Velocity">200</param>
+        <param name="Profile Acceleration">50</param>
+        <param name="Drive Mode">0</param>
+      </gpio>
+      <gpio name="dxl15">
+        <param name="type">dxl</param>
+        <param name="ID">31</param>
+        <command_interface name="Goal Position"/>
+        <state_interface name="Present Position"/>
+        <state_interface name="Present Velocity"/>
+        <!-- <state_interface name="Present Current"/> -->
+        <state_interface name="Torque Enable"/>
+        <state_interface name="Present Input Voltage"/>
+        <param name="Position P Gain">800</param>
+        <!-- <param name="Position I Gain">100</param>
+        <param name="Position D Gain">100</param> -->
+        <param name="Profile Velocity">200</param>
+        <param name="Profile Acceleration">50</param>
+        <!-- <param name="Drive Mode">0</param> -->
       </gpio>
       <gpio name="dxl16">
         <param name="type">dxl</param>
-        <param name="ID">15</param>
-        <command_interface name="Goal Position"/>
-        <state_interface name="Present Position"/>
-        <state_interface name="Present Velocity"/>
-        <state_interface name="Present Current"/>
-        <state_interface name="Torque Enable"/>
-        <state_interface name="Present Input Voltage"/>
-        <param name="Position P Gain">800</param>
-        <param name="Position I Gain">100</param>
-        <param name="Position D Gain">100</param>
-        <param name="Profile Velocity">200</param>
-        <param name="Profile Acceleration">50</param>
-        <param name="Drive Mode">0</param>
-      </gpio> -->
+        <param name="ID">32</param>
+        <command_interface name="Goal Position"/>
+        <state_interface name="Present Position"/>
+        <state_interface name="Present Velocity"/>
+        <!-- <state_interface name="Present Current"/> -->
+        <state_interface name="Torque Enable"/>
+        <state_interface name="Present Input Voltage"/>
+        <param name="Position P Gain">800</param>
+        <!-- <param name="Position I Gain">100</param>
+        <param name="Position D Gain">100</param> -->
+        <param name="Profile Velocity">200</param>
+        <param name="Profile Acceleration">50</param>
+        <!-- <param name="Drive Mode">0</param> -->
+      </gpio>
     </ros2_control>
   </xacro:macro>
