Commit message: kris_moveit_config pkg debug

File: src/kris_moveit_config/config/v2.ros2_control.xacro (robot description, xacro)
@@ -19,41 +19,45 @@
           <param name="error_timeout_sec">0.2</param>
           <param name="dynamixel_model_folder">/param/dxl_model</param>
-          <param name="number_of_joints">16</param>
-          <param name="number_of_transmissions">16</param>
+          <param name="number_of_joints">18</param>
+          <param name="number_of_transmissions">18</param>
           <param name="transmission_to_joint_matrix">
-            1, 0, 0, 0, 0, 0, 0, 0, 0, 0, 0, 0, 0, 0, 0, 0,
-            0, 1, 0, 0, 0, 0, 0, 0, 0, 0, 0, 0, 0, 0, 0, 0,
-            0, 0, 1, 0, 0, 0, 0, 0, 0, 0, 0, 0, 0, 0, 0, 0,
-            0, 0, 0, 1, 0, 0, 0, 0, 0, 0, 0, 0, 0, 0, 0, 0,
-            0, 0, 0, 0, 1, 0, 0, 0, 0, 0, 0, 0, 0, 0, 0, 0,
-            0, 0, 0, 0, 0, 1, 0, 0, 0, 0, 0, 0, 0, 0, 0, 0,
-            0, 0, 0, 0, 0, 0, 1, 0, 0, 0, 0, 0, 0, 0, 0, 0,
-            0, 0, 0, 0, 0, 0, 0, 1, 0, 0, 0, 0, 0, 0, 0, 0,
-            0, 0, 0, 0, 0, 0, 0, 0, 1, 0, 0, 0, 0, 0, 0, 0,
-            0, 0, 0, 0, 0, 0, 0, 0, 0, 1, 0, 0, 0, 0, 0, 0,
-            0, 0, 0, 0, 0, 0, 0, 0, 0, 0, 1, 0, 0, 0, 0, 0,
-            0, 0, 0, 0, 0, 0, 0, 0, 0, 0, 0, 1, 0, 0, 0, 0,
-            0, 0, 0, 0, 0, 0, 0, 0, 0, 0, 0, 0, 1, 0, 0, 0,
-            0, 0, 0, 0, 0, 0, 0, 0, 0, 0, 0, 0, 0, 1, 0, 0,
-            0, 0, 0, 0, 0, 0, 0, 0, 0, 0, 0, 0, 0, 0, 1, 0,
-            0, 0, 0, 0, 0, 0, 0, 0, 0, 0, 0, 0, 0, 0, 0, 1
+            1, 0, 0, 0, 0, 0, 0, 0, 0, 0, 0, 0, 0, 0, 0, 0, 0, 0,
+            0, 1, 0, 0, 0, 0, 0, 0, 0, 0, 0, 0, 0, 0, 0, 0, 0, 0,
+            0, 0, 1, 0, 0, 0, 0, 0, 0, 0, 0, 0, 0, 0, 0, 0, 0, 0,
+            0, 0, 0, 1, 0, 0, 0, 0, 0, 0, 0, 0, 0, 0, 0, 0, 0, 0,
+            0, 0, 0, 0, 1, 0, 0, 0, 0, 0, 0, 0, 0, 0, 0, 0, 0, 0,
+            0, 0, 0, 0, 0, 1, 0, 0, 0, 0, 0, 0, 0, 0, 0, 0, 0, 0,
+            0, 0, 0, 0, 0, 0, 1, 0, 0, 0, 0, 0, 0, 0, 0, 0, 0, 0,
+            0, 0, 0, 0, 0, 0, 0, 1, 0, 0, 0, 0, 0, 0, 0, 0, 0, 0,
+            0, 0, 0, 0, 0, 0, 0, 0, 1, 0, 0, 0, 0, 0, 0, 0, 0, 0,
+            0, 0, 0, 0, 0, 0, 0, 0, 0, 1, 0, 0, 0, 0, 0, 0, 0, 0,
+            0, 0, 0, 0, 0, 0, 0, 0, 0, 0, 1, 0, 0, 0, 0, 0, 0, 0,
+            0, 0, 0, 0, 0, 0, 0, 0, 0, 0, 0, 1, 0, 0, 0, 0, 0, 0,
+            0, 0, 0, 0, 0, 0, 0, 0, 0, 0, 0, 0, 1, 0, 0, 0, 0, 0,
+            0, 0, 0, 0, 0, 0, 0, 0, 0, 0, 0, 0, 0, 1, 0, 0, 0, 0,
+            0, 0, 0, 0, 0, 0, 0, 0, 0, 0, 0, 0, 0, 0, 1, 0, 0, 0,
+            0, 0, 0, 0, 0, 0, 0, 0, 0, 0, 0, 0, 0, 0, 0, 1, 0, 0,
+            0, 0, 0, 0, 0, 0, 0, 0, 0, 0, 0, 0, 0, 0, 0, 0, 1, 0,
+            0, 0, 0, 0, 0, 0, 0, 0, 0, 0, 0, 0, 0, 0, 0, 0, 0, 1
           </param>
           <param name="joint_to_transmission_matrix">
-            1, 0, 0, 0, 0, 0, 0, 0, 0, 0, 0, 0, 0, 0, 0, 0,
-            0, 1, 0, 0, 0, 0, 0, 0, 0, 0, 0, 0, 0, 0, 0, 0,
-            0, 0, 1, 0, 0, 0, 0, 0, 0, 0, 0, 0, 0, 0, 0, 0,
-            0, 0, 0, 1, 0, 0, 0, 0, 0, 0, 0, 0, 0, 0, 0, 0,
-            0, 0, 0, 0, 1, 0, 0, 0, 0, 0, 0, 0, 0, 0, 0, 0,
-            0, 0, 0, 0, 0, 1, 0, 0, 0, 0, 0, 0, 0, 0, 0, 0,
-            0, 0, 0, 0, 0, 0, 1, 0, 0, 0, 0, 0, 0, 0, 0, 0,
-            0, 0, 0, 0, 0, 0, 0, 1, 0, 0, 0, 0, 0, 0, 0, 0,
-            0, 0, 0, 0, 0, 0, 0, 0, 1, 0, 0, 0, 0, 0, 0, 0,
-            0, 0, 0, 0, 0, 0, 0, 0, 0, 1, 0, 0, 0, 0, 0, 0,
-            0, 0, 0, 0, 0, 0, 0, 0, 0, 0, 1, 0, 0, 0, 0, 0,
-            0, 0, 0, 0, 0, 0, 0, 0, 0, 0, 0, 1, 0, 0, 0, 0,
-            0, 0, 0, 0, 0, 0, 0, 0, 0, 0, 0, 0, 1, 0, 0, 0,
-            0, 0, 0, 0, 0, 0, 0, 0, 0, 0, 0, 0, 0, 1, 0, 0,
-            0, 0, 0, 0, 0, 0, 0, 0, 0, 0, 0, 0, 0, 0, 1, 0,
-            0, 0, 0, 0, 0, 0, 0, 0, 0, 0, 0, 0, 0, 0, 0, 1
+            1, 0, 0, 0, 0, 0, 0, 0, 0, 0, 0, 0, 0, 0, 0, 0, 0, 0,
+            0, 1, 0, 0, 0, 0, 0, 0, 0, 0, 0, 0, 0, 0, 0, 0, 0, 0,
+            0, 0, 1, 0, 0, 0, 0, 0, 0, 0, 0, 0, 0, 0, 0, 0, 0, 0,
+            0, 0, 0, 1, 0, 0, 0, 0, 0, 0, 0, 0, 0, 0, 0, 0, 0, 0,
+            0, 0, 0, 0, 1, 0, 0, 0, 0, 0, 0, 0, 0, 0, 0, 0, 0, 0,
+            0, 0, 0, 0, 0, 1, 0, 0, 0, 0, 0, 0, 0, 0, 0, 0, 0, 0,
+            0, 0, 0, 0, 0, 0, 1, 0, 0, 0, 0, 0, 0, 0, 0, 0, 0, 0,
+            0, 0, 0, 0, 0, 0, 0, 1, 0, 0, 0, 0, 0, 0, 0, 0, 0, 0,
+            0, 0, 0, 0, 0, 0, 0, 0, 1, 0, 0, 0, 0, 0, 0, 0, 0, 0,
+            0, 0, 0, 0, 0, 0, 0, 0, 0, 1, 0, 0, 0, 0, 0, 0, 0, 0,
+            0, 0, 0, 0, 0, 0, 0, 0, 0, 0, 1, 0, 0, 0, 0, 0, 0, 0,
+            0, 0, 0, 0, 0, 0, 0, 0, 0, 0, 0, 1, 0, 0, 0, 0, 0, 0,
+            0, 0, 0, 0, 0, 0, 0, 0, 0, 0, 0, 0, 1, 0, 0, 0, 0, 0,
+            0, 0, 0, 0, 0, 0, 0, 0, 0, 0, 0, 0, 0, 1, 0, 0, 0, 0,
+            0, 0, 0, 0, 0, 0, 0, 0, 0, 0, 0, 0, 0, 0, 1, 0, 0, 0,
+            0, 0, 0, 0, 0, 0, 0, 0, 0, 0, 0, 0, 0, 0, 0, 1, 0, 0,
+            0, 0, 0, 0, 0, 0, 0, 0, 0, 0, 0, 0, 0, 0, 0, 0, 1, 0,
+            0, 0, 0, 0, 0, 0, 0, 0, 0, 0, 0, 0, 0, 0, 0, 0, 0, 1
           </param>
           <param name="ros_update_freq">200</param>
@@ -186,4 +190,32 @@
         <state_interface name="velocity"/>
       </joint>
+      <joint name="f18">
+        <command_interface name="position"/>
+        <state_interface name="position">
+          <param name="initial_value">${initial_positions['f18']}</param>
+        </state_interface>
+        <state_interface name="velocity"/>
+      </joint>
+      <!-- <joint name="f19">
+        <command_interface name="position"/>
+        <state_interface name="position">
+          <param name="initial_value">${initial_positions['f19']}</param>
+        </state_interface>
+        <state_interface name="velocity"/>
+      </joint> -->
+      <joint name="f28">
+        <command_interface name="position"/>
+        <state_interface name="position">
+          <param name="initial_value">${initial_positions['f28']}</param>
+        </state_interface>
+        <state_interface name="velocity"/>
+      </joint>
+      <!-- <joint name="f29">
+        <command_interface name="position"/>
+        <state_interface name="position">
+          <param name="initial_value">${initial_positions['f29']}</param>
+        </state_interface>
+        <state_interface name="velocity"/>
+      </joint> -->
       <!-- GPIO Blocks for each dynamixel (IDs 0 to 15 for 16 joints) -->
       <gpio name="dxl1">
@@ -383,4 +415,32 @@
         <param name="Profile Acceleration">50</param>
       </gpio>
+      <gpio name="dxl16">
+        <param name="type">dxl</param>
+        <param name="ID">18</param>
+        <param name="Operating Mode">3</param>
+        <param name="Current Limit">400</param>
+        <command_interface name="Goal Position"/>
+        <state_interface name="Present Position"/>
+        <state_interface name="Present Velocity"/>
+        <state_interface name="Torque Enable"/>
+        <state_interface name="Present Input Voltage"/>
+        <param name="Position P Gain">800</param>
+        <param name="Profile Velocity">200</param>
+        <param name="Profile Acceleration">50</param>
+      </gpio>
+      <gpio name="dxl16">
+        <param name="type">dxl</param>
+        <param name="ID">28</param>
+        <param name="Operating Mode">3</param>
+        <param name="Current Limit">400</param>
+        <command_interface name="Goal Position"/>
+        <state_interface name="Present Position"/>
+        <state_interface name="Present Velocity"/>
+        <state_interface name="Torque Enable"/>
+        <state_interface name="Present Input Voltage"/>
+        <param name="Position P Gain">800</param>
+        <param name="Profile Velocity">200</param>
+        <param name="Profile Acceleration">50</param>
+      </gpio>
     </ros2_control>
   </xacro:macro>

Commit message: add gripper planning groups seperately

File: src/kris_moveit_config/config/v2.ros2_control.xacro (robot description, xacro)
@@ -190,4 +190,5 @@
         <state_interface name="velocity"/>
       </joint>
+      <!-- GRIPPERZZZ -->
       <joint name="f18">
         <command_interface name="position"/>
@@ -197,11 +198,4 @@
         <state_interface name="velocity"/>
       </joint>
-      <!-- <joint name="f19">
-        <command_interface name="position"/>
-        <state_interface name="position">
-          <param name="initial_value">${initial_positions['f19']}</param>
-        </state_interface>
-        <state_interface name="velocity"/>
-      </joint> -->
       <joint name="f28">
         <command_interface name="position"/>
@@ -211,11 +205,4 @@
         <state_interface name="velocity"/>
       </joint>
-      <!-- <joint name="f29">
-        <command_interface name="position"/>
-        <state_interface name="position">
-          <param name="initial_value">${initial_positions['f29']}</param>
-        </state_interface>
-        <state_interface name="velocity"/>
-      </joint> -->
       <!-- GPIO Blocks for each dynamixel (IDs 0 to 15 for 16 joints) -->
       <gpio name="dxl1">
@@ -415,5 +402,6 @@
         <param name="Profile Acceleration">50</param>
       </gpio>
-      <gpio name="dxl16">
+      <!-- GRIPPERZZZ -->
+      <gpio name="dxl17">
         <param name="type">dxl</param>
         <param name="ID">18</param>
@@ -429,5 +417,5 @@
         <param name="Profile Acceleration">50</param>
       </gpio>
-      <gpio name="dxl16">
+      <gpio name="dxl18">
         <param name="type">dxl</param>
         <param name="ID">28</param>

Commit message: j_32 -> j32

File: src/kris_moveit_config/config/v2.ros2_control.xacro (robot description, xacro)
@@ -178,8 +178,8 @@
         <state_interface name="velocity"/>
       </joint>
-      <joint name="j_32">
-        <command_interface name="position"/>
-        <state_interface name="position">
-          <param name="initial_value">${initial_positions['j_32']}</param>
+      <joint name="j32">
+        <command_interface name="position"/>
+        <state_interface name="position">
+          <param name="initial_value">${initial_positions['j32']}</param>
         </state_interface>
         <state_interface name="velocity"/>

File: src/myrobot_description/urdf/v2.urdf (robot description, URDF)
Before this commit: robot v2, 24 links, 23 joints
Joints:
- removed joint j_32
- added joint j32: type revolute, parent neck_yaw, child neck_pitch, origin xyz=0 0.030398 0 rpy=-1.5708 0 1.5708, axis 0 0 1, limit lower=-0.52 upper=0.52 effort=0 velocity=0
